File: PCB/EC23U.kicad_sch (KiCad schematic)
At the start: 24 parts, among them J1 JST, SW1 BOOT0, U1 STM32F401CBUx, U2 XC6206PxxxMR, Y1 8 MHz

Commit message: WIP
Parts:
- added J2: RGB, Connector_PinSocket_2.00mm:PinSocket_1x03_P2.00mm_Vertical, symbol Connector_Generic:Conn_01x03
- added U5: SN74AHCT1G125, Package_TO_SOT_SMD:SOT-23-5, symbol cipulot_parts:SN74AHCT1G125
Connections:
- net +3V3: now also SW1.2 (B); no longer SW1.1 (A)
- net +5V: now also J2.3 (Pin_3), U5.5 (VCC)
- net ADC: no longer U1.10 (PA0), U1.11 (PA1), U1.13 (PA3), U1.14 (PA4), U1.15 (PA5), U1.16 (PA6), U1.17 (PA7), U1.18 (PB0), U1.19 (PB1)
- net AMUX_SEL_0: now also U1.3 (PC14); no longer U1.4 (PC15)
- net AMUX_SEL_1: now also U1.2 (PC13); no longer U1.3 (PC14)
- net AMUX_SEL_2: now also U1.42 (PB6); no longer U1.2 (PC13)
- net APLEX_EN_PIN: now also U1.4 (PC15)
- net BOOT0: now also SW1.1 (A); no longer SW1.2 (B)
- net D+: now also D1.3 (I/O2); no longer D1.2 (I/O1)
- net D-: now also D1.2 (I/O1); no longer D1.3 (I/O2)
- net DISCHARGE_PIN: now also U1.13 (PA3)
- net GND: now also J2.1 (Pin_1), U5.1 (~{OE}), U5.3 (GND)
- net at U1.25 (PB12): now also R5.2
- net at U1.26 (PB13): now also R1.2
- net LED_3V3: now reaches U1.41 (PB5)
- net LED_3V3: now also U5.2 (A)
- net at R4.2: now also U1.17 (PA7)
- net at R2.2: now also U1.18 (PB0)
- new net LED_5V: J2.2 (Pin_2), U5.4 (B)
Other:
- note added: "Header"
- note added: "LED Level Shifter"
- moved on the sheet: C1, R1, R2, R3, R4, R5, U1

Commit message: WIP PCB
Parts:
- added D2: LED, LED_THT:LED_D3.0mm, symbol Device:LED
- added R18: 100, Resistor_SMD:R_0402_1005Metric, symbol Device:R
- J2: footprint Connector_PinSocket_2.00mm:PinSocket_1x03_P2.00mm_Vertical -> Connector_PinSocket_2.54mm:PinSocket_1x03_P2.54mm_Vertical
Connections:
- net GND: now also D2.1 (K)
- net Num_Lock_Led: now reaches U1.27 (PB14)
- net Num_Lock_Led: now also R18.2
- new net: D2.2 (A), R18.1
Other:
- note added: "3.0mm Num Lock LED"
Changed lines of the file:
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@@
   (title_block
     (title "EC23U")
-    (date "2022-11-10")
+    (date "2022-11-11")
     (rev "1")
     (company "Cipulot PCB Design")
@@
     (stroke (width 0) (type default) (color 0 0 0 0))
   )
+  (polyline (pts (xy 57.15 82.55) (xy 81.28 82.55))
+    (stroke (width 0) (type default) (color 0 0 0 0))
+  )
   (polyline (pts (xy 12.7 82.55) (xy 12.7 125.73))
     (stroke (width 0) (type default) (color 0 0 0 0))
@@
     (stroke (width 0) (type default) (color 0 0 0 0))
   )
+  (wire (pts (xy 62.23 100.33) (xy 62.23 100.965))
+    (stroke (width 0) (type default) (color 0 0 0 0))
+  )
   (wire (pts (xy 23.495 31.75) (xy 26.035 31.75))
     (stroke (width 0) (type default) (color 0 0 0 0))
@@
     (stroke (width 0) (type default) (color 0 0 0 0))
   )
+  (wire (pts (xy 118.745 109.855) (xy 122.555 109.855))
+    (stroke (width 0) (type default) (color 0 0 0 0))
+  )
   (wire (pts (xy 118.745 81.915) (xy 122.555 81.915))
     (stroke (width 0) (type default) (color 0 0 0 0))
@@
     (stroke (width 0) (type default) (color 0 0 0 0))
   )
+  (polyline (pts (xy 81.28 82.55) (xy 81.28 119.38))
+    (stroke (width 0) (type default) (color 0 0 0 0))
+  )
   (polyline (pts (xy 78.74 167.64) (xy 85.09 167.64))
     (stroke (width 0) (type default) (color 0 0 0 0))
@@
     (stroke (width 0) (type default) (color 0 0 0 0))
   )
+  (wire (pts (xy 62.23 109.855) (xy 62.23 108.585))
+    (stroke (width 0) (type default) (color 0 0 0 0))
+  )
   (wire (pts (xy 118.745 76.835) (xy 122.555 76.835))
     (stroke (width 0) (type default) (color 0 0 0 0))
@@
   )
   (wire (pts (xy 118.745 89.535) (xy 122.555 89.535))
+    (stroke (width 0) (type default) (color 0 0 0 0))
+  )
+  (wire (pts (xy 62.23 90.805) (xy 62.23 92.71))
     (stroke (width 0) (type default) (color 0 0 0 0))
   )
@@
   )
   (text "Weird Stuff FIx" (at 71.12 162.56 0)
+    (effects (font (size 1.27 1.27)) (justify left bottom))
+  )
+  (text "3.0mm Num Lock LED" (at 58.42 85.725 0)
     (effects (font (size 1.27 1.27)) (justify left bottom))
   )
@@
     )
   )
+  (global_label "Num_Lock_Led" (shape input) (at 62.23 90.805 0) (fields_autoplaced)
+    (effects (font (size 1.27 1.27)) (justify left))
+    (property "Intersheet References" "${INTERSHEET_REFS}" (id 0) (at 78.3107 90.8844 0)
+      (effects (font (size 1.27 1.27)) (justify left) hide)
+    )
+  )
   (global_label "VDD3" (shape input) (at 132.08 177.8 0) (fields_autoplaced)
     (effects (font (size 1.27 1.27)) (justify left))
@@
     (property "Intersheet References" "${INTERSHEET_REFS}" (id 0) (at 24.8444 91.1436 90)
       (effects (font (size 1.27 1.27)) (justify left) hide)
+    )
+  )
+  (global_label "Num_Lock_Led" (shape output) (at 118.745 109.855 180) (fields_autoplaced)
+    (effects (font (size 1.27 1.27)) (justify right))
+    (property "Intersheet References" "${INTERSHEET_REFS}" (id 0) (at 102.6643 109.7756 0)
+      (effects (font (size 1.27 1.27)) (justify right) hide)
     )
   )
@@
     (pin "1")
   )
+  (symbol (lib_id "power:GND") (at 62.23 109.855 0) (unit 1)
+    (in_bom yes) (on_board yes) (fields_autoplaced)
+    (property "Reference" "#PWR052" (id 0) (at 62.23 116.205 0)
+      (effects (font (size 1.27 1.27)) hide)
+    )
+    (property "Value" "GND" (id 1) (at 62.23 114.4175 0))
+    (property "Footprint" "" (id 2) (at 62.23 109.855 0)
+      (effects (font (size 1.27 1.27)) hide)
+    )
+    (property "Datasheet" "" (id 3) (at 62.23 109.855 0)
+      (effects (font (size 1.27 1.27)) hide)
+    )
+    (pin "1")
+  )
+  (symbol (lib_id "Device:LED") (at 62.23 104.775 90) (unit 1)
+    (in_bom yes) (on_board yes) (fields_autoplaced)
+    (property "Reference" "D2" (id 0) (at 65.151 105.5278 90)
+      (effects (font (size 1.27 1.27)) (justify right))
+    )
+    (property "Value" "LED" (id 1) (at 65.151 108.0647 90)
+      (effects (font (size 1.27 1.27)) (justify right))
+    )
+    (property "Footprint" "LED_THT:LED_D3.0mm" (id 2) (at 62.23 104.775 0)
+      (effects (font (size 1.27 1.27)) hide)
+    )
+    (property "Datasheet" "~" (id 3) (at 62.23 104.775 0)
+      (effects (font (size 1.27 1.27)) hide)
+    )
+    (pin "1")
+    (pin "2")
+  )
   (symbol (lib_id "power:+3.3V") (at 277.495 23.495 0) (unit 1)
     (in_bom yes) (on_board yes) (fields_autoplaced)
@@
     (pin "1")
   )
+  (symbol (lib_id "Device:R") (at 62.23 96.52 180) (unit 1)
+    (in_bom yes) (on_board yes)
+    (property "Reference" "R18" (id 0) (at 64.77 96.52 0))
+    (property "Value" "100" (id 1) (at 65.405 98.425 0))
+    (property "Footprint" "Resistor_SMD:R_0402_1005Metric" (id 2) (at 64.008 96.52 90)
+      (effects (font (size 1.27 1.27)) hide)
+    )
+    (property "Datasheet" "~" (id 3) (at 62.23 96.52 0)
+      (effects (font (size 1.27 1.27)) hide)
+    )
+    (property "LCSC" "C25076" (id 4) (at 62.23 96.52 90)
+      (effects (font (size 1.27 1.27)) hide)
+    )
+    (pin "1")
+    (pin "2")
+  )
   (symbol (lib_id "Device:R") (at 114.935 107.315 90) (unit 1)
     (in_bom yes) (on_board yes)
@@
     (property "Reference" "J2" (id 0) (at 92.075 148.0652 0))
     (property "Value" "RGB" (id 1) (at 92.075 150.6021 0))
-    (property "Footprint" "Connector_PinSocket_2.00mm:PinSocket_1x03_P2.00mm_Vertical" (id 2) (at 92.075 155.575 0)
+    (property "Footprint" "Connector_PinSocket_2.54mm:PinSocket_1x03_P2.54mm_Vertical" (id 2) (at 92.075 155.575 0)
       (effects (font (size 1.27 1.27)) hide)
     )
@@
       (reference "#PWR051") (unit 1) (value "GND") (footprint "")
     )
+    (path "/4915c56f-b1a3-4dd1-9b71-525b8d35d698"
+      (reference "#PWR052") (unit 1) (value "GND") (footprint "")
+    )
     (path "/acc9f32a-8c7e-49aa-9351-7dccf232be3b"
       (reference "C1") (unit 1) (value "4.7u") (footprint "Capacitor_SMD:C_0402_1005Metric")
@@
       (reference "D1") (unit 1) (value "PRTR5V0U2X") (footprint "Package_TO_SOT_SMD:SOT-143")
     )
+    (path "/4c4c0b47-6665-46e4-b0a6-fabdb546263f"
+      (reference "D2") (unit 1) (value "LED") (footprint "LED_THT:LED_D3.0mm")
+    )
     (path "/fc9270b8-eadd-43e8-b899-ff5964c1ba96"
       (reference "F1") (unit 1) (value "500mA") (footprint "Fuse:Fuse_0603_1608Metric")
@@
     )
     (path "/f5242914-3abf-465b-9bf0-8fd43b86e5bf"
-      (reference "J2") (unit 1) (value "RGB") (footprint "Connector_PinSocket_2.00mm:PinSocket_1x03_P2.00mm_Vertical")
+      (reference "J2") (unit 1) (value "RGB") (footprint "Connector_PinSocket_2.54mm:PinSocket_1x03_P2.54mm_Vertical")
     )
     (path "/d85b042e-6163-493d-a977-1ddac40ac471"
@@
       (reference "R17") (unit 1) (value "330") (footprint "Capacitor_SMD:C_0402_1005Metric")
     )
+    (path "/d487862d-6e6e-4798-aeae-bfba04d0a05a"
+      (reference "R18") (unit 1) (value "100") (footprint "Resistor_SMD:R_0402_1005Metric")
+    )
     (path "/2d9fc5c6-fdd3-4023-ab91-020570fb26ce"
