File: PCB/analog.kicad_sch (KiCad schematic)
At the start: 13 parts, among them U3 74HC4051, U4 OPA350

Commit message: Update for 3d models
Parts:
- C11, C12: footprint (none) -> Capacitor_SMD:C_0402_1005Metric
- R10, R11, R12, R13, R14, R15, R16, R9: footprint (none) -> Resistor_SMD:R_0402_1005Metric
- U3: footprint (none) -> cipulot_parts:TSSOP16
- U4: footprint (none) -> Package_SO:SOIC-8_3.9x4.9mm_P1.27mm
Changed lines of the file:
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@@
       (effects (font (size 1.27 1.27)) (justify left))
     )
-    (property "Footprint" "" (id 2) (at 52.197 55.245 90)
+    (property "Footprint" "Resistor_SMD:R_0402_1005Metric" (id 2) (at 52.197 55.245 90)
       (effects (font (size 1.27 1.27)) hide)
     )
@@
     (property "Reference" "C12" (id 0) (at 174.625 96.5708 90))
     (property "Value" "100n" (id 1) (at 174.625 94.2594 90))
-    (property "Footprint" "" (id 2) (at 170.815 89.2048 0)
+    (property "Footprint" "Capacitor_SMD:C_0402_1005Metric" (id 2) (at 170.815 89.2048 0)
       (effects (font (size 1.27 1.27)) hide)
     )
@@
       (effects (font (size 1.27 1.27)) (justify left))
     )
-    (property "Footprint" "" (id 2) (at 33.147 55.245 90)
+    (property "Footprint" "Resistor_SMD:R_0402_1005Metric" (id 2) (at 33.147 55.245 90)
       (effects (font (size 1.27 1.27)) hide)
     )
@@
       (effects (font (size 1.524 1.524)))
     )
-    (property "Footprint" "" (id 2) (at 151.765 57.15 0)
+    (property "Footprint" "Package_SO:SOIC-8_3.9x4.9mm_P1.27mm" (id 2) (at 151.765 57.15 0)
       (effects (font (size 1.524 1.524)) hide)
     )
@@
       (effects (font (size 1.27 1.27)) (justify left))
     )
-    (property "Footprint" "" (id 2) (at 26.797 55.245 90)
+    (property "Footprint" "Resistor_SMD:R_0402_1005Metric" (id 2) (at 26.797 55.245 90)
       (effects (font (size 1.27 1.27)) hide)
     )
@@
     (property "Reference" "U3" (id 0) (at 80.645 20.955 0))
     (property "Value" "74HC4051" (id 1) (at 80.645 24.765 0))
-    (property "Footprint" "" (id 2) (at 88.265 48.895 0)
+    (property "Footprint" "cipulot_parts:TSSOP16" (id 2) (at 88.265 48.895 0)
       (effects (font (size 1.27 1.27)) hide)
     )
@@
     (property "Reference" "C11" (id 0) (at 119.9642 77.47 90))
     (property "Value" "220p" (id 1) (at 122.2756 77.47 90))
-    (property "Footprint" "" (id 2) (at 127.3302 81.28 0)
+    (property "Footprint" "Capacitor_SMD:C_0402_1005Metric" (id 2) (at 127.3302 81.28 0)
       (effects (font (size 1.27 1.27)) hide)
     )
@@
       (effects (font (size 1.27 1.27)) (justify left))
     )
-    (property "Footprint" "" (id 2) (at 157.48 83.312 90)
+    (property "Footprint" "Resistor_SMD:R_0402_1005Metric" (id 2) (at 157.48 83.312 90)
       (effects (font (size 1.27 1.27)) hide)
     )
@@
       (effects (font (size 1.27 1.27)) (justify left))
     )
-    (property "Footprint" "" (id 2) (at 64.897 55.245 90)
+    (property "Footprint" "Resistor_SMD:R_0402_1005Metric" (id 2) (at 64.897 55.245 90)
       (effects (font (size 1.27 1.27)) hide)
     )
@@
       (effects (font (size 1.27 1.27)) (justify left))
     )
-    (property "Footprint" "" (id 2) (at 142.367 91.44 90)
+    (property "Footprint" "Resistor_SMD:R_0402_1005Metric" (id 2) (at 142.367 91.44 90)
       (effects (font (size 1.27 1.27)) hide)
     )
@@
       (effects (font (size 1.27 1.27)) (justify left))
     )
-    (property "Footprint" "" (id 2) (at 39.497 55.245 90)
+    (property "Footprint" "Resistor_SMD:R_0402_1005Metric" (id 2) (at 39.497 55.245 90)
       (effects (font (size 1.27 1.27)) hide)
     )
@@
       (effects (font (size 1.27 1.27)) (justify left))
     )
-    (property "Footprint" "" (id 2) (at 45.847 55.245 90)
-      (effects (font (size 1.27 1.27)) hide)
-    )
+    (property "Footprint" "Resistor_SMD:R_0402_1005Metric" (id 2) (at 45.847 55.245 90)
+      (effects (font (size 1.27 1.27)) hide)
+    )
